Commit message: update to com xacro

File: zaber_description/urdf/zaber.ros2_control.xacro (robot description, xacro)
@@ -1,13 +1,13 @@
 <?xml version="1.0"?>
 <robot xmlns:xacro="http://www.ros.org/wiki/xacro">
-  <xacro:macro name="zaber_ros2_control" params="
-    name
-    initial_positions:=${dict(insertion_joint=0.0,horizontal_joint=0.0,vertical_joint=0.0)}
-    ">
+  <xacro:macro name="zaber_ros2_control" params="name
+						 prefix
+						 com_port:=/dev/ttyUSB0">
     <ros2_control name="${name}" type="system">
       <hardware>
         <plugin>zaber_driver/ZaberSystemHardwareInterface</plugin>
+        <param name="com_port">${com_port}</param>
       </hardware>
-      <joint name="horizontal_joint">
+      <joint name="${prefix}horizontal_joint">
         <command_interface name="position">
           <param name="min">-0.05</param>
@@ -18,10 +18,8 @@
           <param name="max"> 0.01</param>
         </command_interface>
-        <state_interface name="position">
-          <!-- initial position for the FakeSystem and simulation -->
-          <param name="initial_value">${initial_positions['horizontal_joint']}</param>
-        </state_interface>
+        <state_interface name="position"/>
+        <state_interface name="velocity"/>
       </joint>
-      <joint name="insertion_joint">
+      <joint name="${prefix}insertion_joint">
         <command_interface name="position">
           <param name="min">0</param>
@@ -32,10 +30,8 @@
           <param name="max"> 0.01</param>
         </command_interface>
-        <state_interface name="position">
-          <!-- initial position for the FakeSystem and simulation -->
-          <param name="initial_value">${initial_positions['insertion_joint']}</param>
-        </state_interface>
+        <state_interface name="position"/>
+        <state_interface name="velocity"/>
       </joint>
-      <joint name="vertical_joint">
+      <joint name="${prefix}vertical_joint">
         <command_interface name="position">
           <param name="min">-0.05</param>
@@ -46,8 +42,6 @@
           <param name="max"> 0.01</param>
         </command_interface>
-        <state_interface name="position">
-          <!-- initial position for the FakeSystem and simulation -->
-          <param name="initial_value">${initial_positions['vertical_joint']}</param>
-        </state_interface>
+        <state_interface name="position"/>
+        <state_interface name="velocity"/>
       </joint>
     </ros2_control>

File: zaber_description/urdf/zaber.urdf.xacro (robot description, xacro)
@@ -1,4 +1,7 @@
 <?xml version="1.0"?>
 <robot xmlns:xacro="http://wiki.ros.org/xacro" name="$(arg name)">
+  <xacro:arg name="name" default="jhu"/>
+  <xacro:arg name="use_ros2_control" default="true"/>
+  <xacro:arg name="com_port" default="/dev/ttyUSB0"/>
   <xacro:include filename="$(find zaber_description)/urdf/zaber_macro.xacro"/>
   <xacro:include filename="$(find zaber_description)/urdf/zaber.ros2_control.xacro"/>
@@ -7,5 +10,7 @@
    <xacro:zaber_robot name="$(arg name)">
    </xacro:zaber_robot>
-   <xacro:zaber_ros2_control name="$(arg name)"/>
+   <xacro:if value="$(arg use_ros2_control)">
+     <xacro:zaber_ros2_control name="$(arg name)" prefix="" com_port="$(arg com_port)"/>
+   </xacro:if>
    <joint name="base_joint" type="fixed">
     <parent link="world"/>
